File: kicad/sheepycam/sheepycam.kicad_pcb (KiCad board)
At the start: 2 copper layers, 11 parts, among them J1 Conn_01x03_Socket, J2 Conn_01x04_Socket, J3 Conn_01x04_Socket, J4 Conn_01x04_Socket, U1 ESP32-WROOM-32D, U2 A4988_STEPPER_MOTOR_DRIVER_CA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, U3 A4988_STEPPER_MOTOR_DRIVER_CA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, U4 A4988_STEPPER_MOTOR_DRIVER_CA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

Commit message: fixed the fucked up repo
Parts:
- removed C1, C2, C3: 100µf, Capacitor_THT:CP_Radial_D5.0mm_P2.00mm
- removed J1: Conn_01x03_Socket, Connector_PinSocket_2.54mm:PinSocket_1x03_P2.54mm_Vertical
- removed J2, J3, J4: Conn_01x04_Socket, Connector_PinSocket_2.54mm:PinSocket_1x04_P2.54mm_Vertical
- removed U1: ESP32-WROOM-32D, ESP32-WROOM-32D:ESP32-WROOMD-Devboard
- added LS1: Active Beeper, Buzzer_Beeper:Buzzer_12x9.5RM7.6, F.Cu at (129.2, 53.8)
- added U5: MCP1825S-3302E/AB, footprints:TO-220_AB_MC_MCH, F.Cu at (118.2, 37.2)
- U2: value A4988_STEPPER_MOTOR_DRIVER_CARRIER -> ~; footprint MODULE_A4988_STEPPER_MOTOR_DRIVER_CARRIER:MODULE_A4988_STEPPER_MOTOR_DRIVER_CARRIER -> Connector_PinHeader_2.54mm:PinHeader_1x06_P2.54mm_Vertical
- U3: value A4988_STEPPER_MOTOR_DRIVER_CARRIER -> ~; footprint MODULE_A4988_STEPPER_MOTOR_DRIVER_CARRIER:MODULE_A4988_STEPPER_MOTOR_DRIVER_CARRIER -> footprints:INMP441
- U4: value A4988_STEPPER_MOTOR_DRIVER_CARRIER -> WeMos_S2_mini; footprint MODULE_A4988_STEPPER_MOTOR_DRIVER_CARRIER:MODULE_A4988_STEPPER_MOTOR_DRIVER_CARRIER -> library:WEMOS_S2_mini
- moved U4 109.2 mm to (84.3, 63.4), turned to 90 degrees
- moved U3 56.3 mm to (118.8, 53.7)
- moved U2 43.4 mm to (112.7, 63.2), turned to 90 degrees
Connections:
- U4 pad 10: unconnected-(U4-VDD-Pad10) -> Net-(U4-GND-Pad10)
- U4 pad 15: Net-(U4-GND-Pad15) -> unconnected-(U4-GPIO37-Pad15)
- U4 pad 9: Net-(U4-GND-Pad15) -> unconnected-(U4-VBUS-Pad9)
