File: kicad/sheepycam/sheepycam.kicad_sch (KiCad schematic)
At the start: 11 parts, among them J1 Conn_01x03_Socket, J2 Conn_01x04_Socket, J3 Conn_01x04_Socket, J4 Conn_01x04_Socket, U1 ESP32-WROOM-32D, U2 A4988_STEPPER_MOTOR_DRIVER_CA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, U3 A4988_STEPPER_MOTOR_DRIVER_CA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, U4 A4988_STEPPER_MOTOR_DRIVER_CA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

Commit message: fixed the fucked up repo
Parts:
- removed C1, C2, C3: 100µf, Capacitor_THT:CP_Radial_D5.0mm_P2.00mm, symbol Device:C_Polarized
- removed J1: Conn_01x03_Socket, Connector_PinSocket_2.54mm:PinSocket_1x03_P2.54mm_Vertical, symbol Connector:Conn_01x03_Socket
- removed J2, J3, J4: Conn_01x04_Socket, Connector_PinSocket_2.54mm:PinSocket_1x04_P2.54mm_Vertical, symbol Connector:Conn_01x04_Socket
- removed U1: ESP32-WROOM-32D, ESP32-WROOM-32D:ESP32-WROOMD-Devboard, symbol ESP32-WROOM-32D:ESP32-WROOM-32D
- removed U2, U3, U4: A4988_STEPPER_MOTOR_DRIVER_CARRIER, MODULE_A4988_STEPPER_MOTOR_DRIVER_CARRIER:MODULE_A4988_STEPPER_MOTOR_DRIVER_CARRIER, symbol A4988_STEPPER_MOTOR_DRIVER_CARRIER:A4988_STEPPER_MOTOR_DRIVER_CARRIER
- added LS1: Active Beeper, Buzzer_Beeper:Buzzer_12x9.5RM7.6, symbol Device:Speaker
- added U1: ~, symbol sheepycam:OV5640
- added U2: ~, Connector_PinHeader_2.54mm:PinHeader_1x06_P2.54mm_Vertical, symbol sheepycam:MicroSd
- added U3: ~, footprints:INMP441, symbol sheepycam:INMP441_Module
- added U4: WeMos_S2_mini, library:WEMOS_S2_mini, symbol s2Mini:WeMos_S2_mini
- added U5: MCP1825S-3302E/AB, footprints:TO-220_AB_MC_MCH, symbol MCP1825S:MCP1825S-3302E_AB
Connections:
- new net: U4.10 (GND), U4.26 (GND)
